Commit message: 基于视觉实现闭环控制

File: urdf/panda_fixed.urdf (robot description, URDF)
Before this commit: robot panda, 13 links, 12 joints
Links:
- added link camera_link, mass 0.1; collision box size=0.02 0.05 0.02; visual box size=0.02 0.05 0.02
- added link camera_link_optical
Joints:
- added joint camera_joint: type fixed, parent panda_hand, child camera_link, origin xyz=0.03 0 0.05 rpy=0.0 -1.57 0.0
- added joint camera_optical_joint: type fixed, parent camera_link, child camera_link_optical, origin xyz=0 0 0 rpy=-1.5708 0 -1.5708
- joint panda_finger_joint2: mimic joint=panda_finger_joint1 -> (none)
